File: zedboard.sch (EAGLE design)
At the start: 24 parts, among them U1 A540Q, U1_C1 0.1u, U1_C2 0.1u

Commit message: finish design
Parts:
- removed J$3: HEARDER_2X1, connectors:HEARDER_2X1
- added CAN1: MKDSN1,5/2-5,08, con-phoenix-508:MKDSN1,5/2-5,08
- added JST1: USB5V, Justin-Eagle-Lib:POWER_CON
- added Q3: BC547, semicon-smd-ipc:NPN-TRANSISTOR_SOT23
- added R10, R9: 1K, rcl:R-EU_R1206
- added R11, R12, R13, R14, R15, R16: 220, rcl:R-EU_R1206
- added SP1: DC-3V, Justin-Eagle-Lib:SPEAKER
- AR1_C1: value (none) -> 0.1u
- J1: value (none) -> Micro-USB
- Q1, Q2: value (none) -> BC547
- R7, R8: value (none) -> 220
- SW1, SW2: value (none) -> 1A125V
Connections:
- removed net N$6: U$2.P$6
- new net N$10: LED1.2+, R15.2
- new net N$11: LED1.1+, R14.2
- new net N$12: LED2.3+, R11.1
- new net N$13: LED2.2+, R12.1
- new net N$14: LED2.1+, R13.1
- new net N$7: Q3.C, R10.1, SP1.-
- new net N$8: Q3.B, R9.2
- new net N$9: LED1.3+, R16.2
- net 3.3V: now also R10.2, SP1.+
- net 5V: now also JST1.V+, R11.2, R12.2, R13.2, R14.1, R15.1, R16.1; no longer J$3.P$1, LED1.1+, LED1.2+, LED1.3+, LED2.1+, LED2.2+, LED2.3+
- net CAN_H: now also CAN1-1.KL
- net CAN_L: now also CAN1-2.KL
- net GND: now also JST1.V-, Q3.E; no longer J$3.P$2
- net SP: now also R9.1
Other:
- moved on the sheet: LED1, LED2
